File: CAD_B/WD1M_BTLE_JDY-08.brd (EAGLE design)
At the start: 25.4 x 36.6 mm, 9 parts, among them J1 CON_HEADER_1X04, Q1 NOFIT_SI2319CDS-T1-GE3

Commit message: adding latest unknown changes
Parts:
- U1: value (none) -> JDY-08JDY-08_MODULE
Connections:
- net D5: now also U1.19; no longer U1.P03/TXDOUT
- net D6: now also U1.20; no longer U1.P02/RXDIN
- net D7: now also U1.22; no longer U1.P00/PWRCN
- net GND: now also U1.24; no longer U1.GND
- net N$11: now also U1.21; no longer U1.P01
- net N$14: now also U1.18; no longer U1.P04/RTCALARMIO
- net N$15: now also U1.17; no longer U1.P05/RTCALARMIO
- net N$16: now also U1.9; no longer U1.P13/IO2
- net N$17: now also U1.10; no longer U1.P15/IO3
- net N$18: now also U1.11; no longer U1.SCK
- net N$19: now also U1.12; no longer U1.SDA
- net N$2: now also U1.23; no longer U1.RSTIN
- net N$20: now also U1.13; no longer U1.P14/IO4
- net N$21: now also U1.14; no longer U1.P10/PWM1
- net N$22: now also U1.15; no longer U1.P07/PWM3
- net N$23: now also U1.16; no longer U1.P06/PWM4
- net N$3: now also U1.2; no longer U1.P22/DEBUGCLOCK
- net N$4: now also U1.3; no longer U1.P21/DEBUGDATA
- net N$5: now also U1.4; no longer U1.P20
- net N$6: now also U1.5; no longer U1.P17
- net N$7: now also U1.6; no longer U1.P16/CONSTATN
- net N$8: now also U1.7; no longer U1.P11/PWM2
- net N$9: now also U1.8; no longer U1.P12/IO1
- net VCC: now also U1.1; no longer U1.VCC_3.3
Other:
- board size 25.4 x 36.6 mm -> 25.4 x 26.8 mm
