File: CAD_B/WD1M_BTLE_JDY-08.sch (EAGLE design)
At the start: 9 parts, among them J1 CON_HEADER_1X04, Q1 NOFIT_SI2319CDS-T1-GE3

Commit message: adding latest unknown changes
Parts:
- U1: value (none) -> JDY-08JDY-08_MODULE; device JDY-08:JDY-08 -> JDY-08:JDY-08JDY-08_MODULE
Other:
- note added: "3.3V POWERED SENSORS: BME280, SHT31 etc"
- note added: "D0 LOW = ON D0 HIGH = OFF"
- note added: "GPIO NUMBERS ARE ARDUINO DIGITAL PINS. D NUMBER ARE NODEMCU PINS. https://escapequotes.net/esp8266-wemos-d1-mini-pins-and-diagram/"
- note added: "GPIO1/TXD0"
- note added: "GPIO3/RXD0"
- note added: "NO FITS ARE OPTIONAL USED FOR DEVELOPMENT PURPOSES."
- note added: "RST ACTIVE ??? ????? ESP8266"
- note added: "WARNING: JDY-08 MODULE DEFAULTS TO 115200 BAUD. SOFTWARE SERIAL IS UNLIKELY TO WORK WITHOUT ERRORS AT THIS SPEED. NEEDS TESTING"
- note removed: "LOW = ON HIGH = OFF"
- note removed: "RST active ??? ????? ESP8266"
- note removed: "RXD0"
- note removed: "SENSORS: BME280, SHT31 etc"
- note removed: "TXD0"
Changed lines of the file:
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@@
 <part name="GND4" library="freetronics-original" deviceset="GND" device=""/>
 <part name="P+2" library="freetronics-original" deviceset="3.3V" device=""/>
-<part name="U1" library="JDY-08" deviceset="JDY-08" device=""/>
+<part name="U1" library="JDY-08" deviceset="JDY-08" device="JDY-08_MODULE"/>
 <part name="Q1" library="SparkFun-DiscreteSemi" deviceset="MOSFET_PCH" device="-IRLML2244" value="NOFIT_SI2319CDS-T1-GE3"/>
 <part name="P+6" library="freetronics-original" deviceset="3.3V" device=""/>
@@
 <text x="228.6" y="104.14" size="1.778" layer="94">GPIO4/SDA</text>
 <text x="228.6" y="106.68" size="1.778" layer="94">GPIO5/SCL</text>
-<text x="228.6" y="109.22" size="1.778" layer="94">RXD0</text>
-<text x="228.6" y="111.76" size="1.778" layer="94">TXD0</text>
+<text x="228.6" y="109.22" size="1.778" layer="94">GPIO3/RXD0</text>
+<text x="228.6" y="111.76" size="1.778" layer="94">GPIO1/TXD0</text>
 <text x="27.94" y="99.06" size="1.778" layer="94" align="bottom-right">GPIO13/MOSI/RXD2</text>
 <text x="27.94" y="104.14" size="1.778" layer="94" align="bottom-right">GPIO14/CLK</text>
@@
 <text x="190.5" y="99.06" size="1.778" layer="97">10k pullup</text>
 <text x="7.62" y="20.32" size="1.778" layer="97">For full D1 Mini specs see http://www.wemos.cc/Products/d1_mini.html</text>
-<text x="25.4" y="165.1" size="1.778" layer="91">RST active ??? ????? ESP8266</text>
-<text x="25.4" y="170.18" size="1.778" layer="91">USING 0805 FOR EASE OF SELF BUILD</text>
+<text x="12.7" y="165.1" size="1.778" layer="91">RST ACTIVE ??? ????? ESP8266</text>
+<text x="12.7" y="167.64" size="1.778" layer="91">USING 0805 FOR EASE OF SELF BUILD</text>
 <text x="157.48" y="83.82" size="1.778" layer="91">TX-&gt;RX
 RX-&gt;TX</text>
 <text x="162.56" y="109.22" size="1.778" layer="91">INTPU</text>
-<text x="83.82" y="45.72" size="1.778" layer="91">LOW = ON
-HIGH = OFF</text>
-<text x="175.26" y="30.48" size="1.778" layer="91">SENSORS: BME280, SHT31 etc</text>
+<text x="73.66" y="45.72" size="1.778" layer="91">D0 LOW = ON
+D0 HIGH = OFF</text>
+<text x="175.26" y="30.48" size="1.778" layer="91">3.3V POWERED SENSORS: BME280, SHT31 etc</text>
+<text x="12.7" y="170.18" size="1.778" layer="91">WARNING: JDY-08 MODULE DEFAULTS TO
+115200 BAUD. SOFTWARE SERIAL IS
+UNLIKELY TO WORK WITHOUT ERRORS
+AT THIS SPEED. NEEDS TESTING</text>
+<text x="12.7" y="162.56" size="1.778" layer="91">NO FITS ARE OPTIONAL USED FOR DEVELOPMENT PURPOSES.</text>
+<text x="12.7" y="154.94" size="1.778" layer="91">GPIO NUMBERS ARE ARDUINO DIGITAL
+PINS. D NUMBER ARE NODEMCU PINS.
+https://escapequotes.net/esp8266-wemos-d1-mini-pins-and-diagram/</text>
 </plain>
 <instances>
